File: pcb/Monotron.sch (KiCad schematic (older format))
At the start: 13 parts, among them J1 DB15_Female_HighDensity, J2 Mini-DIN-6, J3 AudioJack3_Ground, J4 DB9_Male, J5 Conn_02x05_Counter_Clockwise, U1 TivaCLaunchpad

Commit message: Add footprint for capacitor
I actually don't have a capacitor of the required size here right now,
so I'm not sure about the footprint dimensions. However, this footprint
roughly matches the capacitors I do have, and these kinds of THT
footprints shouldn't require much accuracy anyway.
Parts:
- C1: footprint (none) -> Capacitors_THT:C_Disc_D3.4mm_W2.1mm_P2.50mm
Changed lines of the file:
@@
 F 0 "C1" H 3315 6396 50  0000 L CNN
 F 1 "3.3n" H 3315 6305 50  0000 L CNN
-F 2 "" H 3238 6200 50  0001 C CNN
+F 2 "Capacitors_THT:C_Disc_D3.4mm_W2.1mm_P2.50mm" H 3238 6200 50  0001 C CNN
 F 3 "~" H 3200 6350 50  0001 C CNN
 	1    3200 6350

Commit message: Add VGA connector footprint
Parts:
- J1: footprint (none) -> Monotron:ICD15S13E4GX00LF
Changed lines of the file:
@@
 F 0 "J1" H 3200 4717 50  0000 C CNN
 F 1 "DB15_Female_HighDensity" H 3200 4626 50  0000 C CNN
-F 2 "" H 2250 4250 50  0001 C CNN
+F 2 "Monotron:ICD15S13E4GX00LF" H 2250 4250 50  0001 C CNN
 F 3 " ~" H 2250 4250 50  0001 C CNN
 	1    3200 3850

Commit message: Add footprint for PS/2 connector
Parts:
- J2: footprint (none) -> Monotron:5749180-1
Changed lines of the file:
@@
 F 0 "J2" H 6200 1867 50  0000 C CNN
 F 1 "Mini-DIN-6" H 6200 1776 50  0000 C CNN
-F 2 "" H 6200 1500 50  0001 C CNN
+F 2 "Monotron:5749180-1" H 6200 1500 50  0001 C CNN
 F 3 "http://service.powerdynamics.com/ec/Catalog17/Section%2011.pdf" H 6200 1500 50  0001 C CNN
 	1    6200 1500

Commit message: Add footprint for audio connector
Parts:
- J3: footprint (none) -> Monotron:SJ1-3523N
Changed lines of the file:
@@
 F 0 "J3" H 2654 6492 50  0000 C CNN
 F 1 "AudioJack3_Ground" H 2654 6401 50  0000 C CNN
-F 2 "" H 2650 6150 50  0001 C CNN
+F 2 "Monotron:SJ1-3523N" H 2650 6150 50  0001 C CNN
 F 3 "~" H 2650 6150 50  0001 C CNN
 	1    2650 6150

Commit message: Add joystick connector footprint to schematic
Parts:
- J4: footprint (none) -> Monotron:D09P13B4PA00LF
Changed lines of the file:
@@
 F 0 "J4" H 9780 3646 50  0000 L CNN
 F 1 "DB9_Male" H 9780 3555 50  0000 L CNN
-F 2 "" H 9600 3600 50  0001 C CNN
+F 2 "Monotron:D09P13B4PA00LF" H 9600 3600 50  0001 C CNN
 F 3 " ~" H 9600 3600 50  0001 C CNN
 	1    9600 3600

Commit message: Add footprint for jumper cable connector
Parts:
- J5: footprint (none) -> Pin_Headers:Pin_Header_Straight_2x05_Pitch2.54mm
Changed lines of the file:
@@
 F 0 "J5" H 5350 6567 50  0000 C CNN
 F 1 "Conn_02x05_Counter_Clockwise" H 5350 6476 50  0000 C CNN
-F 2 "" H 5300 6150 50  0001 C CNN
+F 2 "Pin_Headers:Pin_Header_Straight_2x05_Pitch2.54mm" H 5300 6150 50  0001 C CNN
 F 3 "~" H 5300 6150 50  0001 C CNN
 	1    5300 6150
