File: pcb/Monotron.kicad_pcb (KiCad board)
At the start: 2 copper layers, 114.3 x 90.2 mm, 13 parts, among them J1 DB15_Female_HighDensity, J2 Mini-DIN-6, J3 AudioJack3_Ground, J4 DB9_Male, J5 Conn_02x05_Counter_Clockwise, U1 TivaCLaunchpad

Commit message: Add credit to PCB
Other:
- outline, holes or cut-outs redrawn
- board text added: "Designed and Manufactured by Braun Robotics https://braun-robotics.com Made in Odenwald"
Changed lines of the file:
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@@
   (general
     (thickness 1.6)
-    (drawings 6)
+    (drawings 7)
     (tracks 125)
     (zones 0)
@@
     )
   )
-  (gr_line (start 152.4 16.51) (end 41.91 16.51) (layer Edge.Cuts) (width 0.15))
+  (gr_line (start 152.4 16.51) (end 43.18 16.51) (layer Edge.Cuts) (width 0.2))
+  (gr_text "Designed and Manufactured by Braun Robotics\nhttps://braun-robotics.com\nMade in Odenwald" (at 129.54 26.67) (layer F.Cu)
+    (effects (font (size 1 1) (thickness 0.2)))
+  )
   (gr_line (start 152.4 19.05) (end 152.4 16.51) (layer Edge.Cuts) (width 0.15))
   (gr_line (start 152.4 106.68) (end 152.4 19.05) (layer Edge.Cuts) (width 0.15))
