File: pcb/monotron.kicad_pcb (KiCad board)
At the start: 2 copper layers, 133.3 x 94 mm, 51 parts, among them J1 Mono / Stereo, J10 DIN5-180, J11 DIN5-180, J12 DE9M, J13 DB25_Female, J14 Mini-DIN-6, J15 Mini-DIN-6, J2 Jack-DC, J3 1x7 Header, J4 AudioJack3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

Commit message: Connect unused inverter inputs to ground.
Connections:
- U3 pad 10: (no net) -> Net-(U3-Pad10)
- U3 pad 11: (no net) -> GND
- U3 pad 12: (no net) -> Net-(U3-Pad12)
- U3 pad 13: (no net) -> GND
Changed lines of the file:
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@@
     (zones 0)
     (modules 51)
-    (nets 123)
+    (nets 125)
   )
   (page A4)
@@
   (layers
     (0 F.Cu signal)
-    (31 B.Cu signal hide)
+    (31 B.Cu signal)
     (32 B.Adhes user hide)
     (33 F.Adhes user)
@@
   (net 121 "Net-(J7-Pad12)")
   (net 122 "Net-(J7-Pad15)")
+  (net 123 "Net-(U3-Pad10)")
+  (net 124 "Net-(U3-Pad12)")
   (net_class Default "This is the default net class."
     (clearance 0.2)
@@
     (add_net "Net-(U1-Pad3.3)")
     (add_net "Net-(U1-Pad3.4)")
+    (add_net "Net-(U3-Pad10)")
+    (add_net "Net-(U3-Pad12)")
     (add_net "Net-(U3-Pad2)")
     (add_net "Net-(U3-Pad5)")
@@
     (pad 3 thru_hole oval (at 0 5.08 90) (size 1.6 1.6) (drill 0.8) (layers *.Cu *.Mask)
       (net 89 "Net-(U3-Pad2)"))
-    (pad 10 thru_hole oval (at 7.62 10.16 90) (size 1.6 1.6) (drill 0.8) (layers *.Cu *.Mask))
+    (pad 10 thru_hole oval (at 7.62 10.16 90) (size 1.6 1.6) (drill 0.8) (layers *.Cu *.Mask)
+      (net 123 "Net-(U3-Pad10)"))
     (pad 4 thru_hole oval (at 0 7.62 90) (size 1.6 1.6) (drill 0.8) (layers *.Cu *.Mask)
       (net 81 "Net-(R12-Pad1)"))
-    (pad 11 thru_hole oval (at 7.62 7.62 90) (size 1.6 1.6) (drill 0.8) (layers *.Cu *.Mask))
+    (pad 11 thru_hole oval (at 7.62 7.62 90) (size 1.6 1.6) (drill 0.8) (layers *.Cu *.Mask)
+      (net 2 GND))
     (pad 5 thru_hole oval (at 0 10.16 90) (size 1.6 1.6) (drill 0.8) (layers *.Cu *.Mask)
       (net 88 "Net-(U3-Pad5)"))
-    (pad 12 thru_hole oval (at 7.62 5.08 90) (size 1.6 1.6) (drill 0.8) (layers *.Cu *.Mask))
+    (pad 12 thru_hole oval (at 7.62 5.08 90) (size 1.6 1.6) (drill 0.8) (layers *.Cu *.Mask)
+      (net 124 "Net-(U3-Pad12)"))
     (pad 6 thru_hole oval (at 0 12.7 90) (size 1.6 1.6) (drill 0.8) (layers *.Cu *.Mask)
       (net 70 "Net-(R13-Pad2)"))
-    (pad 13 thru_hole oval (at 7.62 2.54 90) (size 1.6 1.6) (drill 0.8) (layers *.Cu *.Mask))
+    (pad 13 thru_hole oval (at 7.62 2.54 90) (size 1.6 1.6) (drill 0.8) (layers *.Cu *.Mask)
+      (net 2 GND))
     (pad 7 thru_hole oval (at 0 15.24 90) (size 1.6 1.6) (drill 0.8) (layers *.Cu *.Mask)
       (net 2 GND))
