File: pcb/MIDI_IF.sch (KiCad schematic (older format))
At the start: 14 parts, among them J10 DIN5-180, J11 DIN5-180, J9 DIN5-180, U3 74LS14, U4 6N138

Commit message: Finished adding RTC to PCB layout.
Parts:
- R10, R11, R12, R13, R14, R15: footprint Resistor_THT:R_Axial_DIN0411_L9.9mm_D3.6mm_P12.70mm_Horizontal -> Resistor_THT:R_Axial_DIN0411_L9.9mm_D3.6mm_P5.08mm_Vertical
Connections:
- net at U3.2: now also U3.5; no longer U3.3
- net at U3.4: now also R13.2; no longer R12.1
- net at U3.6: now also R12.1; no longer R13.2
- net at U3.8: now also U3.3; no longer U3.5
Other:
- moved on the sheet: U3B, U3C
Changed lines of the file:
@@
 F 0 "R11" H 3470 4046 50  0000 L CNN
 F 1 "220" H 3470 3955 50  0000 L CNN
-F 2 "Resistor_THT:R_Axial_DIN0411_L9.9mm_D3.6mm_P12.70mm_Horizontal" V 3330 4000 50  0001 C CNN
+F 2 "Resistor_THT:R_Axial_DIN0411_L9.9mm_D3.6mm_P5.08mm_Vertical" V 3330 4000 50  0001 C CNN
 F 3 "~" H 3400 4000 50  0001 C CNN
 	1    3400 4000
@@
 F 0 "R10" H 3470 2246 50  0000 L CNN
 F 1 "220" H 3470 2155 50  0000 L CNN
-F 2 "Resistor_THT:R_Axial_DIN0411_L9.9mm_D3.6mm_P12.70mm_Horizontal" V 3330 2200 50  0001 C CNN
+F 2 "Resistor_THT:R_Axial_DIN0411_L9.9mm_D3.6mm_P5.08mm_Vertical" V 3330 2200 50  0001 C CNN
 F 3 "~" H 3400 2200 50  0001 C CNN
 	1    3400 2200
@@
 F 0 "R14" V 5700 2650 50  0000 C CNN
 F 1 "220" V 5700 2900 50  0000 C CNN
-F 2 "Resistor_THT:R_Axial_DIN0411_L9.9mm_D3.6mm_P12.70mm_Horizontal" V 5730 2750 50  0001 C CNN
+F 2 "Resistor_THT:R_Axial_DIN0411_L9.9mm_D3.6mm_P5.08mm_Vertical" V 5730 2750 50  0001 C CNN
 F 3 "~" H 5800 2750 50  0001 C CNN
 	1    5800 2750
@@
 F 0 "R15" H 7020 3646 50  0000 L CNN
 F 1 "10K" H 7020 3555 50  0000 L CNN
-F 2 "Resistor_THT:R_Axial_DIN0411_L9.9mm_D3.6mm_P12.70mm_Horizontal" V 6880 3600 50  0001 C CNN
+F 2 "Resistor_THT:R_Axial_DIN0411_L9.9mm_D3.6mm_P5.08mm_Vertical" V 6880 3600 50  0001 C CNN
 F 3 "~" H 6950 3600 50  0001 C CNN
 	1    6950 3600
@@
 L 74xx:74LS14 U3
 U 2 1 5C3DE9F6
-P 5300 4200
-F 0 "U3" H 5300 3883 50  0000 C CNN
-F 1 "74LS14" H 5300 3974 50  0000 C CNN
-F 2 "Package_DIP:DIP-14_W7.62mm" H 5300 4200 50  0001 C CNN
-F 3 "http://www.ti.com/lit/gpn/sn74LS14" H 5300 4200 50  0001 C CNN
-	2    5300 4200
+P 5300 2400
+F 0 "U3" H 5300 2083 50  0000 C CNN
+F 1 "74LS14" H 5300 2174 50  0000 C CNN
+F 2 "Package_DIP:DIP-14_W7.62mm" H 5300 2400 50  0001 C CNN
+F 3 "http://www.ti.com/lit/gpn/sn74LS14" H 5300 2400 50  0001 C CNN
+	2    5300 2400
 	-1   0    0    1
 $EndComp
@@
 F 0 "R12" V 4650 4200 50  0000 C CNN
 F 1 "220" V 4750 4200 50  0000 C CNN
-F 2 "Resistor_THT:R_Axial_DIN0411_L9.9mm_D3.6mm_P12.70mm_Horizontal" V 4680 4200 50  0001 C CNN
+F 2 "Resistor_THT:R_Axial_DIN0411_L9.9mm_D3.6mm_P5.08mm_Vertical" V 4680 4200 50  0001 C CNN
 F 3 "~" H 4750 4200 50  0001 C CNN
 	1    4750 4200
@@
 F 0 "R13" V 4950 2450 50  0000 L CNN
 F 1 "220" V 4950 2250 50  0000 L CNN
-F 2 "Resistor_THT:R_Axial_DIN0411_L9.9mm_D3.6mm_P12.70mm_Horizontal" V 4780 2400 50  0001 C CNN
+F 2 "Resistor_THT:R_Axial_DIN0411_L9.9mm_D3.6mm_P5.08mm_Vertical" V 4780 2400 50  0001 C CNN
 F 3 "~" H 4850 2400 50  0001 C CNN
 	1    4850 2400
@@
 L 74xx:74LS14 U3
 U 3 1 5C3DEA42
-P 5300 2400
-F 0 "U3" H 5300 2083 50  0000 C CNN
-F 1 "74LS14" H 5300 2174 50  0000 C CNN
-F 2 "Package_DIP:DIP-14_W7.62mm" H 5300 2400 50  0001 C CNN
-F 3 "http://www.ti.com/lit/gpn/sn74LS14" H 5300 2400 50  0001 C CNN
-	3    5300 2400
+P 5300 4200
+F 0 "U3" H 5300 3883 50  0000 C CNN
+F 1 "74LS14" H 5300 3974 50  0000 C CNN
+F 2 "Package_DIP:DIP-14_W7.62mm" H 5300 4200 50  0001 C CNN
+F 3 "http://www.ti.com/lit/gpn/sn74LS14" H 5300 4200 50  0001 C CNN
+	3    5300 4200
 	-1   0    0    1
 $EndComp

Commit message: Updated Schematic to 0.8.0. (PCB layout still at 0.7.0). Added BOM.
Parts:
- removed unit 6 of U3
- removed unit 5 of U3
- D1: footprint Diode_THT:D_A-405_P12.70mm_Horizontal -> Diode_THT:D_DO-35_SOD27_P7.62mm_Horizontal
- R10, R11, R12, R13, R14, R15: footprint Resistor_THT:R_Axial_DIN0411_L9.9mm_D3.6mm_P5.08mm_Vertical -> Resistor_THT:R_Axial_DIN0204_L3.6mm_D1.6mm_P5.08mm_Horizontal
- R16: footprint Resistor_THT:R_Axial_DIN0411_L9.9mm_D3.6mm_P12.70mm_Horizontal -> Resistor_THT:R_Axial_DIN0204_L3.6mm_D1.6mm_P5.08mm_Horizontal
Connections:
- no-connect marks 9 -> 7
Other:
- moved on the sheet: J9, R10, R13, U3B, U3D
Changed lines of the file:
@@
 Sheet 3 3
 Title "Monotron 32K Schematic"
-Date "2019-01-15"
-Rev "0.7.0"
+Date "2019-02-10"
+Rev "0.8.0"
 Comp "https://github.com/thejpster/monotron"
 Comment1 "Copyright (c) Jonathan 'theJPster' Pallant 2019"
@@
 L Connector:DIN-5_180degree J9
 U 1 1 5C3DE97A
-P 4050 2500
-F 0 "J9" H 4050 2226 50  0000 C CNN
-F 1 "DIN5-180" H 4050 2135 50  0000 C CNN
-F 2 "Monotron:5P180 DIN Socket" H 4050 2500 50  0001 C CNN
-F 3 "https://uk.rs-online.com/web/p/din-connectors/0491087/" H 4050 2500 50  0001 C CNN
-	1    4050 2500
+P 4000 5600
+F 0 "J9" H 4000 5326 50  0000 C CNN
+F 1 "DIN5-180" H 4000 5235 50  0000 C CNN
+F 2 "Monotron:5P180 DIN Socket" H 4000 5600 50  0001 C CNN
+F 3 "https://uk.rs-online.com/web/p/din-connectors/0491087/" H 4000 5600 50  0001 C CNN
+	1    4000 5600
 	1    0    0    -1
 $EndComp
@@
 NoConn ~ 5000 3150
 NoConn ~ 5600 3150
-NoConn ~ 3750 2500
-NoConn ~ 4350 2500
+NoConn ~ 3700 5600
+NoConn ~ 4300 5600
 NoConn ~ 5300 2850
 $Comp
@@
 F 0 "R11" H 3470 4046 50  0000 L CNN
 F 1 "220" H 3470 3955 50  0000 L CNN
-F 2 "Resistor_THT:R_Axial_DIN0411_L9.9mm_D3.6mm_P5.08mm_Vertical" V 3330 4000 50  0001 C CNN
+F 2 "Resistor_THT:R_Axial_DIN0204_L3.6mm_D1.6mm_P5.08mm_Horizontal" V 3330 4000 50  0001 C CNN
 F 3 "~" H 3400 4000 50  0001 C CNN
 	1    3400 4000
@@
 L Device:R R10
 U 1 1 5C3DE9A5
-P 3400 2200
-F 0 "R10" H 3470 2246 50  0000 L CNN
-F 1 "220" H 3470 2155 50  0000 L CNN
-F 2 "Resistor_THT:R_Axial_DIN0411_L9.9mm_D3.6mm_P5.08mm_Vertical" V 3330 2200 50  0001 C CNN
-F 3 "~" H 3400 2200 50  0001 C CNN
-	1    3400 2200
-	1    0    0    -1
-$EndComp
-Wire Wire Line
-	3750 2400 3400 2400
-Wire Wire Line
-	3400 2400 3400 2350
+P 3350 5300
+F 0 "R10" H 3420 5346 50  0000 L CNN
+F 1 "220" H 3420 5255 50  0000 L CNN
+F 2 "Resistor_THT:R_Axial_DIN0204_L3.6mm_D1.6mm_P5.08mm_Horizontal" V 3280 5300 50  0001 C CNN
+F 3 "~" H 3350 5300 50  0001 C CNN
+	1    3350 5300
+	1    0    0    -1
+$EndComp
+Wire Wire Line
+	3700 5500 3350 5500
+Wire Wire Line
+	3350 5500 3350 5450
 $Comp
 L Isolator:6N138 U4
@@
 F 0 "R14" V 5700 2650 50  0000 C CNN
 F 1 "220" V 5700 2900 50  0000 C CNN
-F 2 "Resistor_THT:R_Axial_DIN0411_L9.9mm_D3.6mm_P5.08mm_Vertical" V 5730 2750 50  0001 C CNN
+F 2 "Resistor_THT:R_Axial_DIN0204_L3.6mm_D1.6mm_P5.08mm_Horizontal" V 5730 2750 50  0001 C CNN
 F 3 "~" H 5800 2750 50  0001 C CNN
 	1    5800 2750
@@
 F 0 "D1" V 6000 3050 50  0000 L CNN
 F 1 "1N4148" V 6250 3100 50  0000 L CNN
-F 2 "Diode_THT:D_A-405_P12.70mm_Horizontal" H 6000 3200 50  0001 C CNN
+F 2 "Diode_THT:D_DO-35_SOD27_P7.62mm_Horizontal" H 6000 3200 50  0001 C CNN
 F 3 "~" H 6000 3200 50  0001 C CNN
 	1    6000 3200
@@
 F 0 "R15" H 7020 3646 50  0000 L CNN
 F 1 "10K" H 7020 3555 50  0000 L CNN
-F 2 "Resistor_THT:R_Axial_DIN0411_L9.9mm_D3.6mm_P5.08mm_Vertical" V 6880 3600 50  0001 C CNN
+F 2 "Resistor_THT:R_Axial_DIN0204_L3.6mm_D1.6mm_P5.08mm_Horizontal" V 6880 3600 50  0001 C CNN
 F 3 "~" H 6950 3600 50  0001 C CNN
 	1    6950 3600
@@
 F 0 "R16" H 7220 3146 50  0000 L CNN
 F 1 "470" H 7220 3055 50  0000 L CNN
-F 2 "Resistor_THT:R_Axial_DIN0411_L9.9mm_D3.6mm_P12.70mm_Horizontal" V 7080 3100 50  0001 C CNN
+F 2 "Resistor_THT:R_Axial_DIN0204_L3.6mm_D1.6mm_P5.08mm_Horizontal" V 7080 3100 50  0001 C CNN
 F 3 "~" H 7150 3100 50  0001 C CNN
 	1    7150 3100
@@
 L 74xx:74LS14 U3
 U 2 1 5C3DE9F6
-P 5300 2400
-F 0 "U3" H 5300 2083 50  0000 C CNN
-F 1 "74LS14" H 5300 2174 50  0000 C CNN
-F 2 "Package_DIP:DIP-14_W7.62mm" H 5300 2400 50  0001 C CNN
-F 3 "http://www.ti.com/lit/gpn/sn74LS14" H 5300 2400 50  0001 C CNN
-	2    5300 2400
+P 5300 5500
+F 0 "U3" H 5300 5183 50  0000 C CNN
+F 1 "74LS14" H 5300 5274 50  0000 C CNN
+F 2 "Package_DIP:DIP-14_W7.62mm" H 5300 5500 50  0001 C CNN
+F 3 "http://www.ti.com/lit/gpn/sn74LS14" H 5300 5500 50  0001 C CNN
+	2    5300 5500
 	-1   0    0    1
 $EndComp
@@
 U 1 1 5C3DE9FD
 P 4750 4200
-F 0 "R12" V 4650 4200 50  0000 C CNN
-F 1 "220" V 4750 4200 50  0000 C CNN
-F 2 "Resistor_THT:R_Axial_DIN0411_L9.9mm_D3.6mm_P5.08mm_Vertical" V 4680 4200 50  0001 C CNN
+F 0 "R12" V 4650 4100 50  0000 C CNN
+F 1 "220" V 4650 4300 50  0000 C CNN
+F 2 "Resistor_THT:R_Axial_DIN0204_L3.6mm_D1.6mm_P5.08mm_Horizontal" V 4680 4200 50  0001 C CNN
 F 3 "~" H 4750 4200 50  0001 C CNN
 	1    4750 4200
@@
 L power:GND #PWR0105
 U 1 1 5C3DEA11
-P 4200 2050
-F 0 "#PWR0105" H 4200 1800 50  0001 C CNN
-F 1 "GND" H 4205 1877 50  0000 C CNN
-F 2 "" H 4200 2050 50  0001 C CNN
-F 3 "" H 4200 2050 50  0001 C CNN
-	1    4200 2050
-	1    0    0    -1
-$EndComp
-Wire Wire Line
-	4050 2200 4050 1950
-Wire Wire Line
-	4050 1950 4200 1950
-Wire Wire Line
-	4200 1950 4200 2050
+P 4150 5150
+F 0 "#PWR0105" H 4150 4900 50  0001 C CNN
+F 1 "GND" H 4155 4977 50  0000 C CNN
+F 2 "" H 4150 5150 50  0001 C CNN
+F 3 "" H 4150 5150 50  0001 C CNN
+	1    4150 5150
+	1    0    0    -1
+$EndComp
+Wire Wire Line
+	4000 5300 4000 5050
+Wire Wire Line
+	4000 5050 4150 5050
+Wire Wire Line
+	4150 5050 4150 5150
 $Comp
 L power:+5V #PWR0106
@@
 	7200 4200 7300 4200
 Wire Wire Line
-	6200 2400 6850 2400
-Wire Wire Line
 	7150 2700 7150 2950
 Wire Wire Line
@@
 L Device:R R13
 U 1 1 5C3DEA35
-P 4850 2400
-F 0 "R13" V 4950 2450 50  0000 L CNN
-F 1 "220" V 4950 2250 50  0000 L CNN
-F 2 "Resistor_THT:R_Axial_DIN0411_L9.9mm_D3.6mm_P5.08mm_Vertical" V 4780 2400 50  0001 C CNN
-F 3 "~" H 4850 2400 50  0001 C CNN
-	1    4850 2400
+P 4800 5500
+F 0 "R13" V 4900 5550 50  0000 L CNN
+F 1 "220" V 4900 5350 50  0000 L CNN
+F 2 "Resistor_THT:R_Axial_DIN0204_L3.6mm_D1.6mm_P5.08mm_Horizontal" V 4730 5500 50  0001 C CNN
+F 3 "~" H 4800 5500 50  0001 C CNN
+	1    4800 5500
 	0    -1   -1   0
 $EndComp
@@
 L power:+5V #PWR0108
 U 1 1 5C3DEA3C
-P 3400 2050
-F 0 "#PWR0108" H 3400 1900 50  0001 C CNN
-F 1 "+5V" H 3550 2100 50  0000 C CNN
-F 2 "" H 3400 2050 50  0001 C CNN
-F 3 "" H 3400 2050 50  0001 C CNN
-	1    3400 2050
+P 3350 5150
+F 0 "#PWR0108" H 3350 5000 50  0001 C CNN
+F 1 "+5V" H 3500 5200 50  0000 C CNN
+F 2 "" H 3350 5150 50  0001 C CNN
+F 3 "" H 3350 5150 50  0001 C CNN
+	1    3350 5150
 	1    0    0    -1
 $EndComp
@@
 L 74xx:74LS14 U3
 U 4 1 5C3DEA49
-P 5900 2400
-F 0 "U3" H 5900 2083 50  0000 C CNN
-F 1 "74LS14" H 5900 2174 50  0000 C CNN
-F 2 "Package_DIP:DIP-14_W7.62mm" H 5900 2400 50  0001 C CNN
-F 3 "http://www.ti.com/lit/gpn/sn74LS14" H 5900 2400 50  0001 C CNN
-	4    5900 2400
+P 6050 5500
+F 0 "U3" H 6050 5183 50  0000 C CNN
+F 1 "74LS14" H 6050 5274 50  0000 C CNN
+F 2 "Package_DIP:DIP-14_W7.62mm" H 6050 5500 50  0001 C CNN
+F 3 "http://www.ti.com/lit/gpn/sn74LS14" H 6050 5500 50  0001 C CNN
+	4    6050 5500
 	-1   0    0    1
 $EndComp
@@
 	5650 2750 4950 2750
 Wire Wire Line
-	4350 2400 4700 2400
-Text Notes 4250 2700 0    50   ~ 0
+	4300 5500 4650 5500
+Text Notes 3850 6100 0    50   ~ 0
 MIDI Out
-Text Notes 4850 3350 0    50   ~ 0
+Text Notes 5150 3650 0    50   ~ 0
 MIDI In
-Text Notes 3350 4450 0    50   ~ 0
+Text Notes 3800 4800 0    50   ~ 0
 MIDI Through
-$Comp
-L 74xx:74LS14 U3
-U 6 1 5C3DEA59
-P 9100 4700
-F 0 "U3" V 9050 4750 50  0000 R CNN
-F 1 "74LS14" V 8900 4650 50  0000 R CNN
-F 2 "" H 9100 4700 50  0001 C CNN
-F 3 "http://www.ti.com/lit/gpn/sn74LS14" H 9100 4700 50  0001 C CNN
-	6    9100 4700
-	0    -1   -1   0
-$EndComp
 $Comp
 L 74xx:74LS14 U?
@@
 Wire Wire Line
 	9450 3600 9450 3650
-$Comp
-L 74xx:74LS14 U?
-U 5 1 5C3F4C23
-P 9600 4700
-AR Path="/5C3F4C23" Ref="U?"  Part="5"
-AR Path="/5C3C82B1/5C3F4C23" Ref="U3"  Part="5"
-F 0 "U3" V 9550 4750 50  0000 R CNN
-F 1 "74LS14" V 9400 4650 50  0000 R CNN
-F 2 "" H 9600 4700 50  0001 C CNN
-F 3 "http://www.ti.com/lit/gpn/sn74LS14" H 9600 4700 50  0001 C CNN
-	5    9600 4700
-	0    -1   -1   0
-$EndComp
-$Comp
-L power:GND #PWR?
-U 1 1 5C3F4C2A
-P 9600 5000
-AR Path="/5C526519/5C3F4C2A" Ref="#PWR?"  Part="1"
-AR Path="/5C3F4C2A" Ref="#PWR?"  Part="1"
-AR Path="/5C3C82B1/5C3F4C2A" Ref="#PWR0110"  Part="1"
-F 0 "#PWR0110" H 9600 4750 50  0001 C CNN
-F 1 "GND" H 9605 4827 50  0000 C CNN
-F 2 "" H 9600 5000 50  0001 C CNN
-F 3 "" H 9600 5000 50  0001 C CNN
-	1    9600 5000
-	1    0    0    -1
-$EndComp
-$Comp
-L power:GND #PWR?
-U 1 1 5C3F4C30
-P 9100 5000
-AR Path="/5C526519/5C3F4C30" Ref="#PWR?"  Part="1"
-AR Path="/5C3F4C30" Ref="#PWR?"  Part="1"
-AR Path="/5C3C82B1/5C3F4C30" Ref="#PWR0111"  Part="1"
-F 0 "#PWR0111" H 9100 4750 50  0001 C CNN
-F 1 "GND" H 9105 4827 50  0000 C CNN
-F 2 "" H 9100 5000 50  0001 C CNN
-F 3 "" H 9100 5000 50  0001 C CNN
-	1    9100 5000
-	1    0    0    -1
-$EndComp
-Text HLabel 6850 2400 2    50   Input ~ 0
+Text HLabel 6800 5500 2    50   Input ~ 0
 MCU_TO_MIDI
 Text HLabel 7000 4350 0    50   Output ~ 0
@@
 Wire Wire Line
 	7200 4200 7200 4350
-NoConn ~ 9600 4400
-NoConn ~ 9100 4400
+Wire Wire Line
+	5600 5500 5750 5500
+Wire Wire Line
+	6350 5500 6800 5500
+Wire Wire Line
+	4950 5500 5000 5500
 $EndSCHEMATC
