File: pcb/monotron.sch (KiCad schematic (older format))
At the start: 43 parts, among them J1 1x3 Header, J12 DE9M, J16 Micro_SD_Card_Det, J2 2.1mm DC Jack, J3 DNF, J4 3.5mm TRS Jack, J5 DE9M, J6 1x4 Header, J7 DE15HD, J8 2x6 Header, U1 TM4C123G_Launchpad, U2 MAX3232, U6 MCP7940N-xP, Y1 32,768 kHz

Commit message: Tidied up schematic.
Parts:
- removed J2: 2.1mm DC Jack, Connector_BarrelJack:BarrelJack_CUI_PJ-102AH_Horizontal, symbol Connector:Jack-DC
- added C1, C14, C7, C8: 100n, Capacitor_THT:C_Disc_D5.0mm_W2.5mm_P2.50mm, symbol Device:C
- added D2: 1N4148, Diode_THT:D_DO-35_SOD27_P7.62mm_Horizontal, symbol Device:D
- added J1: 2.1mm DC Jack, symbol Connector:Jack-DC
- added J12, J13: Mini-DIN-6, Monotron:mini-DIN 6, symbol Connector:Mini-DIN-6
- added J14: DB25_Female, Connector_Dsub:DSUB-25_Male_Horizontal_P2.77x2.84mm_EdgePinOffset7.70mm_Housed_MountingHolesOffset9.12mm, symbol Connector:DB25_Female
- added J4, J5, J6: DIN5-180, Monotron:5P180 DIN Socket, symbol Connector:DIN-5_180degree
- added J8: 2x3 Header, symbol Connector_Generic:Conn_02x03_Odd_Even
- added R1: 470, Resistor_THT:R_Axial_DIN0204_L3.6mm_D1.6mm_P5.08mm_Horizontal, symbol Device:R
- added R10, R6, R7, R8, R9: 220, Resistor_THT:R_Axial_DIN0204_L3.6mm_D1.6mm_P5.08mm_Horizontal, symbol Device:R
- added R2: 10K, Resistor_THT:R_Axial_DIN0204_L3.6mm_D1.6mm_P5.08mm_Horizontal, symbol Device:R
- added U1: 74LS14, Package_DIP:DIP-14_W7.62mm, symbol 74xx:74LS14
- added U2: 6N138, Package_DIP:DIP-8_W7.62mm, symbol Isolator:6N138
- added U5: ATmega48A-PU, Package_DIP:DIP-28_W7.62mm, symbol MCU_Microchip_ATmega:ATmega48A-PU
- renumbered C5 to C10, C8 to C11, C9 to C12, C10 to C13, C1 to C15, C2 to C16, C7 to C17, C3 to C2, C17 to C3, C15 to C4, C16 to C5, C4 to C9, D2 to D1, J1 to J10, J12 to J11, J7 to J15, J3 to J17, J5 to J2, J6 to J3, J8 to J7, J4 to J9, R3 to R11, R4 to R12, R1 to R13, R2 to R14, R7 to R15, R8 to R16, R9 to R17, R17 to R18, R18 to R19, R19 to R20, R20 to R21, R21 to R3, R5 to R4, R6 to R5, U6 to U3, U1 to U4, U2 to U6
Connections:
- net labels added: ACK, AUTOF, BUSY, D0, D1, D2, D3_MOSI, D4_MISO, D5_SCK, D6, D7, ERROR, INIT, KB_CLK, KB_DATA, MS_CLK, MS_DATA, PB2_INIT, PE, SEL, SELPRIN, STROBE
- net labels removed: DCD, DSR, DTE_CTS, DTE_RTS, DTE_RX, DTE_TX, DTR, PB2_LPT_INIT, RI
- wire segments 230 -> 377
- no-connect marks 27 -> 38
Other:
- note added: "5V INPUT"
- note added: "AUDIO OUTPUT"
- note added: "Atmel ISP Header\nUnplug printer first!"
- note added: "I/O EXPANDER"
- note added: "JOYSTICK INPUT"
- note added: "Keyboard"
- note added: "LEVEL SHIFTER"
- note added: "MAIN PROCESSOR BOARD"
- note added: "MIDI INTERFACE"
- note added: "MIDI In"
- note added: "MIDI Out"
- note added: "MIDI Through"
- note added: "Mouse"
- note added: "PARALLEL PRINTER INTERFACE"
- note added: "PS/2 INTERFACES"
- note added: "Parallel\nPrinter Port"
- note added: "REAL TIME CLOCK"
- note added: "RS-232 INTERFACE"
- note added: "Remove jumpers and\nattach 3.3V FTDI cable.\nNot 5V-tolerant!\nDO NOT SUPPLY 3.3V HERE!"
- note added: "SD CARD INTERFACES"
- note added: "The Atmel is one pin short, so we drive nINIT\nfrom the MCU, using these hex inverters\nas a level shifter"
- note added: "VGA OUTPUT"
- note removed: "Atari Joystick"
- note removed: "Power Input"
- note removed: "RS232"
- note removed: "Remove jumpers and\nattach 3.3V FTDI cable.\nNot 5V-tolerant!"
- note removed: "VGA Video"
- moved on the sheet: BT1, C10, C11, C12, C13, C15, C16, C17, C2, C3, C4, C5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

Commit message: WIP re-laying out board.
Parts:
- added D3: D_TVS, Diode_THT:D_5W_P12.70mm_Horizontal, symbol Device:D_TVS
- added F1: Polyfuse, Capacitor_THT:C_Disc_D7.5mm_W4.4mm_P5.00mm, symbol Device:Polyfuse
- added H1: DP14085, Monotron:DP14085, symbol Mechanical:MountingHole
- C15, C16, C2: symbol Device:C -> Device:CP
- J1: footprint (none) -> Connector_BarrelJack:BarrelJack_CUI_PJ-102AH_Horizontal
- J8: footprint (none) -> Connector_PinHeader_2.54mm:PinHeader_2x03_P2.54mm_Vertical
- U4: footprint Launchpad:Launchpad_4x10 -> Monotron:Launchpad_4x10; Digikey 296-35760-ND -> 609-6378-ND‎
Connections:
- net labels added: LPT_ACK, LPT_AUTOF, LPT_BUSY, LPT_D0, LPT_D1, LPT_D2, LPT_D3_MOSI, LPT_D4_MISO, LPT_D5_SCK, LPT_D6, LPT_D7, LPT_ERROR, LPT_INIT, LPT_PE, LPT_SEL, LPT_SELPRIN, LPT_STROBE, PB3_NC, PD1_PB6_NC
- net labels removed: ACK, AUTOF, BUSY, D0, D1, D2, D3_MOSI, D4_MISO, D5_SCK, D6, D7, ERROR, INIT, PB3_SPARE, PB6_SPARE, PE, SEL, SELPRIN, STROBE
- wire segments 377 -> 376
Other:
- note added: "AtMega USART Input"
- note added: "AtMega USART Output"
- note added: "TVS trips at 6.4V\nPolyFuse passes 500mA, trips at 1A"
- note added: "Wired as DTE"
- moved on the sheet: C1, C11, C14, C6, C7, C8, D1, D2, J1, J4, J5, R1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
