File: pcb/monotron.sch (KiCad schematic (older format))
At the start: 68 parts, among them J1 2.1mm DC Jack, J10 1x3 Header, J11 DE9M, J12 Mini-DIN-6, J13 Mini-DIN-6, J14 DB25_Female, J15 DE15HD, J16 Micro_SD_Card_Det, J17 DNF, J2 DE9M, J3 1x4 Header, J4 DIN5-180, J5 DIN5-180, J6 DIN5-180, J7 2x6 Header, J8 2x3 Header, J9 3.5mm TRS Jack, U1 74LS14, U2 6N138, U3 MCP7940N-xP, U4 TM4C123G_Launchpad, U5 ATmega48A-PU, U6 MAX3232, Y1 32,768 kHz

Commit message: Added two Megadrive ports, USB power, and extra SPI ports.
Parts:
- removed J1: 2.1mm DC Jack, Connector_BarrelJack:BarrelJack_CUI_PJ-102AH_Horizontal, symbol Connector:Jack-DC
- added C20, C3, C4: 10u, Capacitor_THT:C_Radial_D5.0mm_H5.0mm_P2.00mm, symbol Device:CP
- added J1: USB_B_Micro, symbol Connector:USB_B_Micro
- added J3: DE9M, Connector_Dsub:DSUB-9_Male_Horizontal_P2.77x2.84mm_EdgePinOffset7.70mm_Housed_MountingHolesOffset9.12mm, symbol Connector:DB9_Male
- added U3: MCP23017_SP, Package_DIP:DIP-28_W7.62mm, symbol Interface_Expansion:MCP23017_SP
- C2: value 47u -> 220u
- renumbered C9 to C10, C10 to C11, C7 to C14, C8 to C18, C14 to C19, C3 to C5, C4 to C6, C5 to C7, C6 to C8, C11 to C9, D3 to D1, D1 to D3, J9 to J10, J10 to J11, J11 to J12, J12 to J13, J13 to J14, J14 to J15, J15 to J16, J16 to J17, J17 to J18, J5 to J4, J4 to J5, J3 to J7, J7 to J8, J8 to J9, R8 to R1, R1 to R4, R4 to R5, R5 to R6, R6 to R7, R7 to R8, U3 to U5, U5 to U6, U6 to U7
Connections:
- net labels added: JS1_DOWN, JS1_FIRE1, JS1_FIRE2, JS1_LEFT, JS1_RIGHT, JS1_SELECT, JS1_UP, JS2_DOWN, JS2_FIRE1, JS2_FIRE2, JS2_LEFT, JS2_RIGHT, JS2_SELECT, JS2_UP, PA2_SPI_CLK, PA3_SPI_CS1, PA4_SPI_MISO, PA5_SPI_MOSI, PD7_SPI_CS3, PF4_SPI_CS2, ~ATMEGA_RESET
- net labels removed: PA2_SD_CLK, PA3_SD_CS, PA4_SD_MISO, PA5_SD_MOSI, PB3_NC, PD1_PB6_NC, PD6_JS_LEFT, PD7_JS_RIGHT, PE2_JS_UP, PE3_JS_DOWN, PF4_JS_FIRE
- wire segments 376 -> 421
- no-connect marks 38 -> 49
Other:
- note added: "I2C Expansion EEEEEEEE\nMove to this to couple of SPI/I2C expansion port\nSite them near the PCB edge so they can take an SPI WiFi/LAN module"
- note added: "JOYSTICK INPUTS"
- note removed: "I2C Expansion"
- note removed: "JOYSTICK INPUT"
- moved on the sheet: BT1, C2, C5, C6, C7, D1, F1, J2, J7, J9, U5, Y1

Commit message: Add expansion headers.
Parts:
- removed J7: 1x4 Header, Connector_PinHeader_2.54mm:PinHeader_1x04_P2.54mm_Vertical, symbol Connector:Conn_01x04_Male
- added J?: Expansion A, symbol Connector_Generic:Conn_02x08_Counter_Clockwise
- added J?: Expansion B, symbol Connector_Generic:Conn_02x08_Counter_Clockwise
Connections:
- net labels added: JS1_0, JS1_1, JS1_2, JS1_3, JS1_A, JS1_B, JS1_SEL, JS2_0, JS2_1, JS2_2, JS2_3, JS2_A, JS2_B, JS2_SEL, PA3_SPI_CS0, PB3_SPI_CS2, PD6_U2RX, PD7_U2TX, PF4_SPI_CS1, RS232_BUS
- net labels removed: JS1_DOWN, JS1_FIRE1, JS1_FIRE2, JS1_LEFT, JS1_RIGHT, JS1_SELECT, JS1_UP, JS2_DOWN, JS2_FIRE1, JS2_FIRE2, JS2_LEFT, JS2_RIGHT, JS2_SELECT, JS2_UP, PA3_SPI_CS1, PD7_SPI_CS3, PF4_SPI_CS2
- wire segments 421 -> 446
- no-connect marks 49 -> 46
Other:
- note added: "Designed for Sparkfun BOB-00544\nFit J17 or J18 - not both"
- note added: "EXPANSION (UART 2, SPI 1+2, I2C)"
- note added: "Expansion Slots A and B\nModules can use UART, SPI or I2C\nUART only supported on Expansion A"
- note added: "I/O EXPANDER (UART 7)"
- note added: "JOYSTICK INPUTS (I2C)"
- note added: "MIDI INTERFACE (UART 3)"
- note added: "REAL TIME CLOCK (I2C)"
- note added: "RS-232 INTERFACE (UART 1)"
- note added: "SD CARD INTERFACES (SPI 0)"
- note added: "SMT micro-SD\nFit J17 or J18 - not both\n"
- note removed: "Fit Sparkfun BOB-00544"
- note removed: "I/O EXPANDER"
- note removed: "I2C Expansion EEEEEEEE\nMove to this to couple of SPI/I2C expansion port\nSite them near the PCB edge so they can take an SPI WiFi/LAN module"
- note removed: "JOYSTICK INPUTS"
- note removed: "MIDI INTERFACE"
- note removed: "REAL TIME CLOCK"
- note removed: "RS-232 INTERFACE"
- note removed: "SD CARD INTERFACES"
- note removed: "SMT micro-SD"
- moved on the sheet: BT1, C1, C10, C11, C12, C13, C15, C16, C17, C20, C4, C5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
