File: pcb/tiva_mcu/tivac_mcu.sch (KiCad schematic (older format))
At the start: 23 parts, among them J1 USB Power, J2 3.5mm TRS Jack, J3 1x3 Header, J4 DE15HD, J5 Monotron_Bridge_MCU_Side, U1 TM4C123G_Launchpad

Commit message: Working on new PCB design - ATX format.
Parts:
- J5: footprint Connector_PinHeader_2.54mm:PinHeader_2x32_P2.54mm_Horizontal -> Connector_PinSocket_2.54mm:PinSocket_2x24_P2.54mm_Horizontal
Connections:
- net labels added: AUD_L, AUD_R, BLU, GRN, RED
- wire segments 214 -> 175
Other:
- moved on the sheet: J2, R5, R6, RN1
